File: docs/resources/physbryk_power_supply/physbryk_power_supply.kicad_pcb (KiCad board)
At the start: 2 copper layers, 50.8 x 72.4 mm, 12 parts, among them U1 LM317_TO-220

Commit message: added kicad files for the power supply
Parts:
- MES1: value Voltmeter_DC_LED -> Volt_Ammeter
Connections:
- MES1 pad 2: Net-(H1-Pad1) -> Net-(MES1-Pad2)
- MES1 pad 3: Net-(BT1-Pad1) -> Net-(H1-Pad1)
- R1 pad 2: Net-(H1-Pad1) -> Net-(MES1-Pad2)
- U1 pad 2: Net-(H1-Pad1) -> Net-(MES1-Pad2)
Routing:
- net Net-(MES1-Pad2): track 0.00 -> 29.5 mm
- net Net-(H1-Pad1): track 63.7 -> 49.5 mm
- net Net-(BT1-Pad1): track 32.7 -> 28.5 mm
