File: docs/cad/physbryk_feather/physbryk_feather.kicad_pcb (KiCad board)
At the start: 2 copper layers, 50.8 x 22.9 mm, 5 parts, among them J1 Conn_01x04_Male, SW1 SW_SPDT

Commit message: added kicad gerbers
Connections:
- JP1 pad 11: Net-(J1-Pad3) -> Net-(J1-Pad1)
- JP1 pad 12: Net-(J1-Pad4) -> Net-(J1-Pad2)
- JP3 pad 13: Net-(J1-Pad1) -> Net-(J1-Pad4)
- JP3 pad 14: Net-(J1-Pad2) -> Net-(JP3-Pad14)
- JP3 pad 15: Net-(JP3-Pad15) -> Net-(J1-Pad3)
- MS1 pad 17: Net-(J1-Pad4) -> Net-(J1-Pad2)
- MS1 pad 18: Net-(J1-Pad3) -> Net-(J1-Pad1)
- MS1 pad 2: Net-(JP3-Pad15) -> Net-(J1-Pad3)
- MS1 pad 3: Net-(J1-Pad2) -> Net-(JP3-Pad14)
- MS1 pad 4: Net-(J1-Pad1) -> Net-(J1-Pad4)
- SW1 pad 2: Net-(J1-Pad1) -> Net-(J1-Pad4)
Routing:
- net Net-(J1-Pad4): track 7.14 -> 51.9 mm
- net Net-(J1-Pad1): track 49.4 -> 15.2 mm
- net Net-(J1-Pad3): track 10.2 -> 41.8 mm
- net Net-(J1-Pad2): track 38.4 -> 12.3 mm
- net Net-(JP3-Pad15): track 2.54 -> 0.00 mm
- net Net-(JP3-Pad14): track 0.00 -> 2.54 mm
